Commit message: lidar 3d fixed

File: urdf/diy_ackermann.urdf.xacro (robot description, xacro)
@@ -281,9 +281,16 @@
   <!-- LiDAR 3D - Tarea -->
   <joint type="fixed" name="lidar_joint_gazebo">
-    <origin xyz="0 0 0.035" rpy="0 0 0"/>
+    <origin xyz="0 0 0.095" rpy="0 0 0"/>
     <child link="lidar_link_gazebo" />
     <parent link="chassis"/>
   </joint>
   <link name="lidar_link_gazebo">
+    <visual>
+      <origin xyz="0 0 0" rpy="0 0 0"/>
+      <geometry>
+        <cylinder length="0.15" radius="0.075"/>
+      </geometry>
+      <material name="blue"/>
+    </visual>
     <inertial>
       <mass value="0.1"/>
@@ -293,5 +300,5 @@
       <origin xyz="0 0 0.0" rpy="0 0 0"/>
       <geometry>
-        <cylinder length="0.07" radius="0.04"/>
+        <cylinder length="0.15" radius="0.075"/>
       </geometry>
     </collision>
@@ -304,5 +311,5 @@
     <sensor name='ouster_lidar' type='gpu_lidar'>
       <topic>/robot/lidar</topic>
-      <gz_frame_id>chassis</gz_frame_id>
+      <gz_frame_id>lidar_link_gazebo</gz_frame_id>
       <update_rate>10</update_rate>
       <lidar>
@@ -322,6 +329,6 @@
         </scan>
         <range>
-          <min>0.08</min>
-          <max>100.0</max>
+          <min>0.1</min>
+          <max>30.0</max>
           <resolution>0.01</resolution>
         </range>
@@ -424,3 +431,6 @@
     <material>Gazebo/Red</material>
   </gazebo>
+  <gazebo reference="lidar_link_gazebo">
+    <material>Gazebo/Blue</material>
+  </gazebo>
 </robot>

Commit message: readme updated

File: urdf/diy_ackermann.urdf.xacro (robot description, xacro)
@@ -280,65 +280,69 @@
   </joint>
   <!-- LiDAR 3D - Tarea -->
-  <joint type="fixed" name="lidar_joint_gazebo">
-    <origin xyz="0 0 0.095" rpy="0 0 0"/>
-    <child link="lidar_link_gazebo" />
+  <!-- 1. Propiedades del sensor -->
+  <xacro:property name="lidar3d_size" value="0.15"/>
+  <xacro:property name="lidar3d_mass" value="0.8"/>
+  <!-- 2. Link del LiDAR 3D -->
+  <link name="lidar_3d_link">
+    <visual>
+      <origin xyz="0 0 0" rpy="0 0 0"/>
+      <geometry>
+        <cylinder radius="${lidar3d_size/2}" length="${lidar3d_size}"/>
+      </geometry>
+      <material name="blue"/>
+    </visual>
+    <collision>
+      <origin xyz="0 0 0" rpy="0 0 0"/>
+      <geometry>
+        <cylinder radius="${lidar3d_size/2}" length="${lidar3d_size}"/>
+      </geometry>
+    </collision>
+    <xacro:cylinder_inertia mass="${lidar3d_mass}"
+                            radius="${lidar3d_size/2}"
+                            height="${lidar3d_size}"/>
+  </link>
+  <joint name="lidar_3d_joint" type="fixed">
+    <origin xyz="0 0 ${chassis_height/2 + lidar3d_size + 0.05}" rpy="0 0 0"/>
     <parent link="chassis"/>
-  </joint>
-  <link name="lidar_link_gazebo">
-    <visual>
-      <origin xyz="0 0 0" rpy="0 0 0"/>
-      <geometry>
-        <cylinder length="0.15" radius="0.075"/>
-      </geometry>
-      <material name="blue"/>
-    </visual>
-    <inertial>
-      <mass value="0.1"/>
-      <inertia ixx="0.001" ixy="0.0" ixz="0.0" iyy="0.001" iyz="0.0" izz="0.001"/>
-    </inertial>
-    <collision name="collision-base">
-      <origin xyz="0 0 0.0" rpy="0 0 0"/>
-      <geometry>
-        <cylinder length="0.15" radius="0.075"/>
-      </geometry>
-    </collision>
-  </link>
+    <child link="lidar_3d_link"/>
+  </joint>
   <!-- ========================================== -->
   <!-- GAZEBO PLUGINS -->
   <!-- ========================================== -->
   <!-- LiDAR 3D Plugin -->
-  <gazebo reference="lidar_link_gazebo">
-    <sensor name='ouster_lidar' type='gpu_lidar'>
-      <topic>/robot/lidar</topic>
-      <gz_frame_id>lidar_link_gazebo</gz_frame_id>
+  <gazebo reference="lidar_3d_link">
+  <sensor name="lidar_3d" type="gpu_lidar">  <!-- Cambiar a type="lidar" si no tienes GPU -->
+    <topic>lidar_3d</topic>
+    <gz_frame_id>lidar_3d_link</gz_frame_id>
       <update_rate>10</update_rate>
-      <lidar>
-        <scan>
-          <horizontal>
-            <samples>1024</samples>
-            <resolution>1.0</resolution>
-            <min_angle>-3.1415926</min_angle>
-            <max_angle>3.1415926</max_angle>
-          </horizontal>
-          <vertical>
-            <samples>32</samples>
-            <resolution>1</resolution>
-            <min_angle>-0.39</min_angle>
-            <max_angle>0.39</max_angle>
-          </vertical>
-        </scan>
-        <range>
-          <min>0.1</min>
-          <max>30.0</max>
-          <resolution>0.01</resolution>
-        </range>
-        <noise type="gaussian">
-          <mean>0.0</mean>
-          <stddev>0.01</stddev>
-        </noise>
-      </lidar>
-      <alwaysOn>1</alwaysOn>
-      <visualize>true</visualize>
-    </sensor>
+    <lidar>
+      <scan>
+        <horizontal>
+          <samples>1800</samples>
+          <resolution>1</resolution>
+          <min_angle>-3.14159</min_angle>
+          <max_angle>3.14159</max_angle>
+        </horizontal>
+        <vertical>
+          <samples>16</samples>
+          <resolution>1</resolution>
+          <min_angle>-0.2617</min_angle>  <!-- -15° -->
+          <max_angle>0.2617</max_angle>   <!-- +15° -->
+        </vertical>
+      </scan>
+      <range>
+        <min>0.5</min>
+        <max>30.0</max>
+        <resolution>0.01</resolution>
+      </range>
+      <noise>
+        <type>gaussian</type>
+        <mean>0.0</mean>
+        <stddev>0.02</stddev>
+      </noise>
+    </lidar>
+    <always_on>1</always_on>
+    <visualize>true</visualize>
+  </sensor>
   </gazebo>
   <!-- Ackermann Drive Plugin -->
